File: hardware/mainboard/Top.kicad_sch (KiCad schematic)
At the start: 0 parts

Commit message: latest
Other:
- added sheet eigeneSchaltungserweiterungen (untitled.kicad_sch)
- note removed: "${##}"
- note removed: "${#}"
- note removed: "${BOARD_ASSEMBLY_REVISION}"
- note removed: "${BOARD_DOCUMENT_DATE}"
- note removed: "${BOARD_NAME}"
- note removed: "${BOARD_PCB_REVISION}"
- note removed: "${BOARD_REFERENCE}"
- note removed: "${TITLE}"
- note removed: "${VARIANTNAME}"
- note removed: "-"
- note removed: "A4"
- note removed: "Date:"
- note removed: "Project:"
- note removed: "Reference:"
- note removed: "Revision:"
- note removed: "Sheet:"
- note removed: "Size:"
- note removed: "Title:"
- note removed: "Variant:"
- note removed: "of"
